File: Garden PCB/Garden PCB.kicad_pcb (KiCad board)
At the start: 2 copper layers, 250 x 100 mm, 87 parts, among them IC1 LM74500QDDFRQ1, J1 GPIO, J10 Conn_02x05_Odd_Even, J11 Screw_Terminal_01x10, J12 Screw_Terminal_01x02, J2 Conn_02x06_Top_Bottom, J3 Conn_02x05_Odd_Even, J4 Conn_02x05_Odd_Even, J5 Conn_02x05_Odd_Even, J6 Conn_02x05_Odd_Even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

Commit message: fixes for power switch, also looks like KiCad might have boned some of our pinouts
Parts:
- removed the C5 at (230.9, 116.3)
- added C11: .1uf, RCER71H104K0DBH03A:RCER71H104K0DBH03A, F.Cu at (231.0, 116.4)
- RV1: value MOV-14D201KKTR -> V14E14AUTO
- SW1: footprint M2011SS1W01:M2011SS1W01CUL -> 7105SYV3QE:7105SYV3QE
- moved IC1 12.1 mm to (175.1, 148.2)
- moved Q1 12.1 mm to (168.9, 145.4)
- moved VCAP1 12.1 mm to (178.5, 148.4)
- moved C6 9.70 mm to (169.3, 155.5), turned to 0 degrees
- moved SW1 5.77 mm to (219.1, 164.1)
- moved TVS1 4.78 mm to (169.8, 162.1), turned to 0 degrees
- moved RV1 3.60 mm to (189.2, 164.8)
- moved F1 3.13 mm to (207.1, 164.5)
- moved C8 1.49 mm to (162.3, 135.4)
Connections:
- IC1 pad 4: Net-(IC1-VCAP) -> GND
- IC1 pad 5: Net-(IC1-EN) -> Net-(IC1-SOURCE)
- VCAP1 pad 1: Net-(IC1-EN) -> Net-(IC1-SOURCE)
- VCAP1 pad 2: Net-(IC1-VCAP) -> GND
Routing:
- net GND: track 554.7 -> 472.5 mm, vias 3 -> 0
- net Net-(J12-Pin_1): track 8.62 -> 20.7 mm
- net Net-(SW1-B): track 16.6 -> 25.5 mm
- net Net-(IC1-EN): track 37.1 -> 29.5 mm
- net Net-(C6-Pad1): track 62.6 -> 67.6 mm
- net +12V: track 489.6 -> 492.8 mm
- net Net-(IC1-VCAP): track 2.36 -> 0.00 mm
- net Net-(IC1-SOURCE): track 0.00 -> 1.96 mm
